File: examples/simple.kicad_pcb (KiCad board)
At the start: 2 copper layers, 40 x 20 mm, 3 parts

Commit message: Add KiCad placement round trip
Parts:
- removed ? (x2): , terminal
- removed ?: , obstacle
- added H1: , obstacle, F.Cu at (20.0, 10.0)
- added J1: , terminal, F.Cu at (5.00, 10.0)
- added J2: , terminal, F.Cu at (35.0, 10.0)
Changed lines of the file:
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@@
   (net 1 "SIGNAL")
   (footprint "terminal" (layer "F.Cu") (at 5 10)
+    (fp_text reference "J1" (at 0 0) (layer "F.Fab") hide)
     (pad "1" thru_hole circle (at 0 0) (size 1.5 1.5) (drill 0.8) (layers "*.Cu" "*.Mask") (net 1 "SIGNAL")))
   (footprint "terminal" (layer "F.Cu") (at 35 10)
+    (fp_text reference "J2" (at 0 0) (layer "F.Fab") hide)
     (pad "1" thru_hole circle (at 0 0) (size 1.5 1.5) (drill 0.8) (layers "*.Cu" "*.Mask") (net 1 "SIGNAL")))
   (footprint "obstacle" (layer "F.Cu") (at 20 10)
+    (fp_text reference "H1" (at 0 0) (layer "F.Fab") hide)
     (pad "" np_thru_hole rect (at 0 0) (size 8 14) (drill 3) (layers "*.Cu" "*.Mask")))
   (gr_rect (start 0 0) (end 40 20) (stroke (width 0.05) (type default)) (fill none) (layer "Edge.Cuts"))
