File: examples/multilayer.kicad_pcb (KiCad board)
At the start: 4 copper layers, 40 x 20 mm, 4 parts

Commit message: feat: generate reproducible manufacturing packages (#429)
Generate deterministic, hash-bound Gerber, drill, BOM, CPL, DRC, and manifest artifacts from isolated staged KiCad projects. Harden metadata validation and output publication, and cover KiCad 10 multilayer behavior with end-to-end tests.
Parts:
- J1, J2: value (none) -> TEST_POINT
Changed lines of the file:
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@@
   (general (thickness 1.6))
   (paper "A4")
-  (layers (0 "F.Cu" signal) (2 "In1.Cu" signal) (4 "In2.Cu" signal) (31 "B.Cu" signal) (44 "Edge.Cuts" user))
+  (layers (0 "F.Cu" signal) (2 "In1.Cu" signal) (4 "In2.Cu" signal) (31 "B.Cu" signal)
+    (32 "B.Paste" user "b.paste") (33 "F.Paste" user "f.paste")
+    (34 "B.Mask" user "b.mask") (35 "F.Mask" user "f.mask")
+    (36 "B.SilkS" user "b.silkscreen") (37 "F.SilkS" user "f.silkscreen")
+    (44 "Edge.Cuts" user))
   (setup (pad_to_mask_clearance 0))
   (net 0 "")
@@
   (footprint "terminal" (layer "F.Cu") (at 5 10)
     (fp_text reference "J1" (at 0 0) (layer "F.Fab") hide)
-    (pad "1" smd circle (at 0 0) (size 1.5 1.5) (layers "F.Cu") (net 1 "SIGNAL")))
+    (fp_text value "TEST_POINT" (at 0 1) (layer "F.Fab") hide)
+    (property "LCSC Part #" "C-LIVE-1")
+    (pad "1" smd circle (at 0 0) (size 1.5 1.5) (layers "F.Cu" "F.Paste" "F.Mask") (net 1 "SIGNAL")))
   (footprint "terminal" (layer "F.Cu") (at 35 10)
     (fp_text reference "J2" (at 0 0) (layer "F.Fab") hide)
-    (pad "1" smd circle (at 0 0) (size 1.5 1.5) (layers "F.Cu") (net 1 "SIGNAL")))
+    (fp_text value "TEST_POINT" (at 0 1) (layer "F.Fab") hide)
+    (property "LCSC Part #" "C-LIVE-1")
+    (pad "1" smd circle (at 0 0) (size 1.5 1.5) (layers "F.Cu" "F.Paste" "F.Mask") (net 1 "SIGNAL")))
   (footprint "front-obstacle" (layer "F.Cu") (at 20 10)
     (fp_text reference "O1" (at 0 0) (layer "F.Fab") hide)
+    (attr exclude_from_bom exclude_from_pos_files)
     (pad "" smd rect (at 0 0) (size 8 18) (layers "F.Cu")))
   (footprint "back-obstacle" (layer "B.Cu") (at 20 10)
     (fp_text reference "O2" (at 0 0) (layer "B.Fab") hide)
+    (attr exclude_from_bom exclude_from_pos_files)
     (pad "" smd rect (at 0 0) (size 8 18) (layers "B.Cu")))
   (gr_rect (start 0 0) (end 40 20) (stroke (width 0.05) (type default)) (fill none) (layer "Edge.Cuts"))
